File: onekey_remote/mops-out.kicad_pcb (KiCad board)
At the start: 2 copper layers, 56.5 x 53 mm, 28 parts, among them CN1 AFC12-S02CCC-00, J1 microusb, J2 tradfri_debugger, Q1 2N7002, SW1 Toggle, SW2 reset, U1 TRADFRI, U2 AP131-33, U3 BL8573CB6TR

Commit message: readme
Changed lines of the file:
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@@
       (drillshape 0)
       (scaleselection 1)
-      (outputdirectory "tradfri/"))
+      (outputdirectory "mops-tradfri/"))
   )
   (net 0 "")
@@
     (fp_line (start 1.85 0.95) (end 1.85 -0.95) (layer B.CrtYd) (width 0.05))
     (fp_line (start 1.85 -0.95) (end -1.85 -0.95) (layer B.CrtYd) (width 0.05))
-    (pad 2 smd roundrect (at 1.025 0 220) (size 1.15 1.4) (layers B.Cu B.Paste B.Mask) (roundrect_rratio 0.217391)
+    (pad 2 smd roundrect (at 1.025 0 220) (size 1.15 1.4) (layers B.Cu B.Paste B.Mask) (roundrect_rratio 0.2173904347826087)
       (net 31 "Net-(D6-Pad2)"))
-    (pad 1 smd roundrect (at -1.025 0 220) (size 1.15 1.4) (layers B.Cu B.Paste B.Mask) (roundrect_rratio 0.217391)
+    (pad 1 smd roundrect (at -1.025 0 220) (size 1.15 1.4) (layers B.Cu B.Paste B.Mask) (roundrect_rratio 0.2173904347826087)
       (net 18 PC10))
     (model ${KISYS3DMOD}/LED_SMD.3dshapes/LED_0805_2012Metric.wrl
@@
     (fp_line (start 1.85 0.95) (end 1.85 -0.95) (layer B.CrtYd) (width 0.05))
     (fp_line (start 1.85 -0.95) (end -1.85 -0.95) (layer B.CrtYd) (width 0.05))
-    (pad 2 smd roundrect (at 1.025 0 300) (size 1.15 1.4) (layers B.Cu B.Paste B.Mask) (roundrect_rratio 0.217391)
-      (net 9 +3V3))
-    (pad 1 smd roundrect (at -1.025 0 300) (size 1.15 1.4) (layers B.Cu B.Paste B.Mask) (roundrect_rratio 0.217391)
+    (pad 2 smd roundrect (at 1.025 0 300) (size 1.15 1.4) (layers B.Cu B.Paste B.Mask) (roundrect_rratio 0.2173904347826087)
+      (net 9 +3V3))
+    (pad 1 smd roundrect (at -1.025 0 300) (size 1.15 1.4) (layers B.Cu B.Paste B.Mask) (roundrect_rratio 0.2173904347826087)
       (net 28 "Net-(D3-Pad1)"))
     (model ${KISYS3DMOD}/LED_SMD.3dshapes/LED_0805_2012Metric.wrl
@@
     (fp_line (start 1.85 0.95) (end 1.85 -0.95) (layer B.CrtYd) (width 0.05))
     (fp_line (start 1.85 -0.95) (end -1.85 -0.95) (layer B.CrtYd) (width 0.05))
-    (pad 2 smd roundrect (at 1.025 0 180) (size 1.15 1.4) (layers B.Cu B.Paste B.Mask) (roundrect_rratio 0.217391)
-      (net 9 +3V3))
-    (pad 1 smd roundrect (at -1.025 0 180) (size 1.15 1.4) (layers B.Cu B.Paste B.Mask) (roundrect_rratio 0.217391)
+    (pad 2 smd roundrect (at 1.025 0 180) (size 1.15 1.4) (layers B.Cu B.Paste B.Mask) (roundrect_rratio 0.2173904347826087)
+      (net 9 +3V3))
+    (pad 1 smd roundrect (at -1.025 0 180) (size 1.15 1.4) (layers B.Cu B.Paste B.Mask) (roundrect_rratio 0.2173904347826087)
       (net 28 "Net-(D3-Pad1)"))
     (model ${KISYS3DMOD}/LED_SMD.3dshapes/LED_0805_2012Metric.wrl
@@
     (fp_line (start 1.85 0.95) (end 1.85 -0.95) (layer B.CrtYd) (width 0.05))
     (fp_line (start 1.85 -0.95) (end -1.85 -0.95) (layer B.CrtYd) (width 0.05))
-    (pad 2 smd roundrect (at 1.025 0 60) (size 1.15 1.4) (layers B.Cu B.Paste B.Mask) (roundrect_rratio 0.217391)
-      (net 9 +3V3))
-    (pad 1 smd roundrect (at -1.025 0 60) (size 1.15 1.4) (layers B.Cu B.Paste B.Mask) (roundrect_rratio 0.217391)
+    (pad 2 smd roundrect (at 1.025 0 60) (size 1.15 1.4) (layers B.Cu B.Paste B.Mask) (roundrect_rratio 0.2173904347826087)
+      (net 9 +3V3))
+    (pad 1 smd roundrect (at -1.025 0 60) (size 1.15 1.4) (layers B.Cu B.Paste B.Mask) (roundrect_rratio 0.2173904347826087)
       (net 28 "Net-(D3-Pad1)"))
     (model ${KISYS3DMOD}/LED_SMD.3dshapes/LED_0805_2012Metric.wrl
