File: onekey_remote/mops-out.sch (KiCad schematic (older format))
At the start: 26 parts, among them CN1 AFC12-S02CCC-00, J1 microusb, Q1 2N7002, SW1 Toggle, SW2 reset, U2 AP131-33, U3 BL8573CB6TR

Commit message: readme
Parts:
- D1: value LED -> red
- D2: value LED -> green
Changed lines of the file:
@@
 P 4650 6000
 F 0 "D2" H 4643 6217 50  0000 C CNN
-F 1 "LED" H 4643 6126 50  0000 C CNN
+F 1 "green" H 4643 6126 50  0000 C CNN
 F 2 "LED_SMD:LED_0603_1608Metric_Pad1.05x0.95mm_HandSolder" H 4650 6000 50  0001 C CNN
 F 3 "~" H 4650 6000 50  0001 C CNN
@@
 P 2850 5900
 F 0 "D1" H 2843 5645 50  0000 C CNN
-F 1 "LED" H 2843 5736 50  0000 C CNN
+F 1 "red" H 2843 5736 50  0000 C CNN
 F 2 "LED_SMD:LED_0603_1608Metric_Pad1.05x0.95mm_HandSolder" H 2850 5900 50  0001 C CNN
 F 3 "~" H 2850 5900 50  0001 C CNN
