File: onekey_remote_cr2032/mops-out.kicad_pcb (KiCad board)
At the start: 2 copper layers, 56.5 x 53 mm, 19 parts, among them J2 tradfri_debugger, Q1 2N7002, SW1 Toggle, SW2 reset, U1 TRADFRI

Commit message: pcb
Parts:
- moved SW2 0.50 mm to (145.5, 48.6)
Routing:
- net GND: track 157.3 -> 155.5 mm
Other:
- outline, holes or cut-outs redrawn
Changed lines of the file:
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@@
     (thickness 1.6)
     (drawings 46)
-    (tracks 209)
+    (tracks 212)
     (zones 0)
     (modules 19)
@@
   )
   (module mybays_connector:KEY_ALPS_SKRTLBE010 (layer F.Cu)
-    (at 145 48.6 180)
+    (at 145.5 48.6 180)
     (fp_text reference SW2 (at 3.114107 4.424365) (layer F.SilkS)
       (effects (font (size 1 1) (thickness 0.15)))
@@
       (net 1 GND))
   )
+  (gr_circle (center 145.8468 91.98356) (end 146.32432 92.22994) (layer Edge.Cuts) (width 0.05))
   (gr_arc (start 102 98) (end 100 98) (angle -90) (layer Edge.Cuts) (width 0.05))
   (gr_arc (start 154.5 98) (end 154.5 100) (angle -90) (layer Edge.Cuts) (width 0.05))
   (gr_arc (start 154.5 49) (end 156.5 49) (angle -90) (layer Edge.Cuts) (width 0.05))
-  (gr_circle (center 145.86 91.33) (end 146.36 91.33) (layer Edge.Cuts) (width 0.05))
   (gr_line (start 104 96) (end 104 61) (layer F.SilkS) (width 0.12))
   (gr_line (start 104 96) (end 152.5 96) (layer F.SilkS) (width 0.12))
@@
   (gr_line (start 100 65) (end 118 65) (layer F.SilkS) (width 0.12))
   (gr_line (start 100 65.5) (end 118 65.5) (layer F.SilkS) (width 0.12))
-  (gr_line (start 133 47) (end 133 53) (layer F.SilkS) (width 0.05))
-  (gr_line (start 133 53) (end 139 53) (layer F.SilkS) (width 0.05))
-  (gr_line (start 139 53) (end 139 47) (layer F.SilkS) (width 0.05))
+  (gr_line (start 134 47) (end 134 53) (layer F.SilkS) (width 0.05))
+  (gr_line (start 134 53) (end 140 53) (layer F.SilkS) (width 0.05))
+  (gr_line (start 140 53) (end 140 47) (layer F.SilkS) (width 0.05))
   (gr_line (start 147.5 47) (end 147.5 50) (layer F.SilkS) (width 0.05))
   (gr_line (start 147.5 50) (end 143.5 50) (layer F.SilkS) (width 0.05))
@@
   (gr_circle (center 128.25 75) (end 128.25 99) (layer B.SilkS) (width 0.12))
   (gr_circle (center 128.25 75) (end 128.25 99.9) (layer B.SilkS) (width 0.12))
-  (gr_circle (center 105 96) (end 105 97.15) (layer Edge.Cuts) (width 0.05))
+  (gr_circle (center 105.1 96) (end 106.25 96) (layer Edge.Cuts) (width 0.05))
   (gr_circle (center 151.5 96) (end 151.5 97.15) (layer Edge.Cuts) (width 0.05))
-  (gr_circle (center 151.5 58) (end 151.5 59.15) (layer Edge.Cuts) (width 0.05))
-  (gr_circle (center 120.1 50) (end 120.1 51.15) (layer Edge.Cuts) (width 0.05))
-  (gr_circle (center 103 67.5) (end 103 68.65) (layer Edge.Cuts) (width 0.05))
+  (gr_circle (center 151.5 57.9) (end 152.65 57.9) (layer Edge.Cuts) (width 0.05))
+  (gr_circle (center 120.2 49.9) (end 121.35 49.9) (layer Edge.Cuts) (width 0.05))
+  (gr_circle (center 102.9 67.5) (end 104.05 67.5) (layer Edge.Cuts) (width 0.05))
   (gr_line (start 102 100) (end 154.5 100) (layer Edge.Cuts) (width 0.05))
   (gr_line (start 156.5 98) (end 156.5 91) (layer Edge.Cuts) (width 0.05))
@@
   (gr_line (start 102.5 92) (end 100 92) (layer Edge.Cuts) (width 0.05))
   (gr_line (start 100 92) (end 100 98) (layer Edge.Cuts) (width 0.05))
-  (segment (start 143.784356 48.247194) (end 143.09627 47.559108) (width 0.65) (layer F.Cu) (net 1))
-  (segment (start 143.784356 49.640638) (end 143.784356 48.247194) (width 0.65) (layer F.Cu) (net 1))
-  (segment (start 146.18618 48.276912) (end 146.90373 47.559362) (width 0.65) (layer F.Cu) (net 1))
-  (segment (start 146.18618 49.640638) (end 146.18618 48.276912) (width 0.65) (layer F.Cu) (net 1))
-  (segment (start 142.800106 47.855272) (end 143.09627 47.559108) (width 0.65) (layer F.Cu) (net 1))
-  (segment (start 142.800106 48.6) (end 142.800106 47.855272) (width 0.65) (layer F.Cu) (net 1))
-  (segment (start 147.199894 47.855526) (end 146.90373 47.559362) (width 0.65) (layer F.Cu) (net 1))
-  (segment (start 147.199894 48.6) (end 147.199894 47.855526) (width 0.65) (layer F.Cu) (net 1))
-  (segment (start 147.0025 50.456958) (end 146.18618 49.640638) (width 0.35) (layer F.Cu) (net 1))
-  (segment (start 147.0025 52.89) (end 147.0025 50.456958) (width 0.35) (layer F.Cu) (net 1))
   (segment (start 143.096524 47.559362) (end 143.09627 47.559108) (width 0.35) (layer F.Cu) (net 1))
-  (segment (start 146.90373 47.559362) (end 143.096524 47.559362) (width 0.35) (layer F.Cu) (net 1))
   (segment (start 124.89993 73.149991) (end 131.10007 73.149991) (width 0.65) (layer B.Cu) (net 1))
   (segment (start 115.57 91.27998) (end 115.57 97.029778) (width 0.65) (layer F.Cu) (net 1))
@@
   (segment (start 117.908999 61.694001) (end 117.908999 60.912499) (width 0.35) (layer F.Cu) (net 1))
   (segment (start 120.584 60.944) (end 119.758999 61.769001) (width 0.35) (layer F.Cu) (net 1))
-  (segment (start 142.800106 50.224064) (end 142.800106 48.6) (width 0.35) (layer B.Cu) (net 1))
   (segment (start 135.636 57.38817) (end 142.800106 50.224064) (width 0.35) (layer B.Cu) (net 1))
   (segment (start 135.636 58.547) (end 135.636 57.38817) (width 0.35) (layer B.Cu) (net 1))
@@
   (segment (start 130.556 72.605921) (end 131.10007 73.149991) (width 0.35) (layer B.Cu) (net 1))
   (segment (start 130.556 71.12) (end 130.556 72.605921) (width 0.35) (layer B.Cu) (net 1))
+  (segment (start 142.800106 49.1) (end 143.300106 48.6) (width 0.35) (layer B.Cu) (net 1))
+  (segment (start 142.800106 50.224064) (end 142.800106 49.1) (width 0.35) (layer B.Cu) (net 1))
+  (segment (start 143.59627 48.303836) (end 143.300106 48.6) (width 0.35) (layer F.Cu) (net 1))
+  (segment (start 143.59627 47.559108) (end 143.59627 48.303836) (width 0.35) (layer F.Cu) (net 1))
+  (segment (start 144.284356 49.58425) (end 143.300106 48.6) (width 0.35) (layer F.Cu) (net 1))
+  (segment (start 144.284356 49.640638) (end 144.284356 49.58425) (width 0.35) (layer F.Cu) (net 1))
+  (segment (start 147.40373 48.303836) (end 147.699894 48.6) (width 0.35) (layer F.Cu) (net 1))
+  (segment (start 147.40373 47.559362) (end 147.40373 48.303836) (width 0.35) (layer F.Cu) (net 1))
+  (segment (start 147.699894 48.626924) (end 146.68618 49.640638) (width 0.35) (layer F.Cu) (net 1))
+  (segment (start 147.699894 48.6) (end 147.699894 48.626924) (width 0.35) (layer F.Cu) (net 1))
+  (segment (start 146.68618 52.57368) (end 147.0025 52.89) (width 0.35) (layer F.Cu) (net 1))
+  (segment (start 146.68618 49.640638) (end 146.68618 52.57368) (width 0.35) (layer F.Cu) (net 1))
+  (segment (start 147.403476 47.559108) (end 147.40373 47.559362) (width 0.35) (layer F.Cu) (net 1))
+  (segment (start 143.59627 47.559108) (end 147.403476 47.559108) (width 0.35) (layer F.Cu) (net 1))
   (segment (start 138.176 58.547) (end 139.27699 58.547) (width 0.35) (layer B.Cu) (net 2))
   (segment (start 139.27699 58.547) (end 140.41999 59.69) (width 0.35) (layer B.Cu) (net 2))
@@
   (segment (start 128.27 62.665894) (end 128.27 78.109002) (width 0.35) (layer F.Cu) (net 8))
   (segment (start 144.985268 52.597768) (end 145.2775 52.89) (width 0.25) (layer F.Cu) (net 11))
-  (segment (start 144.985268 49.640638) (end 144.985268 52.597768) (width 0.25) (layer F.Cu) (net 11))
   (segment (start 152.047944 79.478124) (end 154.81602 76.710048) (width 0.35) (layer F.Cu) (net 11))
   (segment (start 154.81602 66.381719) (end 145.796 57.361699) (width 0.35) (layer F.Cu) (net 11))
@@
   (segment (start 145.796 53.4085) (end 145.2775 52.89) (width 0.35) (layer F.Cu) (net 11))
   (segment (start 145.796 57.361699) (end 145.796 53.4085) (width 0.35) (layer F.Cu) (net 11))
+  (segment (start 145.485268 52.682232) (end 145.2775 52.89) (width 0.35) (layer F.Cu) (net 11))
+  (segment (start 145.485268 49.640638) (end 145.485268 52.682232) (width 0.35) (layer F.Cu) (net 11))
   (segment (start 149.787478 75.5885) (end 149.697948 75.67803) (width 0.35) (layer F.Cu) (net 13))
   (segment (start 153.416 75.5885) (end 149.787478 75.5885) (width 0.35) (layer F.Cu) (net 13))
